Commit message: Configure 6-drone area coverage simulation, optimal RRA return sweeps, and Gazebo 3D support

File: urdf/drone.urdf (robot description, URDF)
Before this commit: robot drone, 4 links, 3 joints
Links:
- link base_link: geometry collision box size=0.4 0.4 0.12; visual box size=0.25 0.03 0.02

Commit message: Configure 6-drone area coverage simulation, optimal RRA return sweeps, and Gazebo 3D support

File: urdf/drone.urdf (robot description, URDF)
Before this commit: robot drone, 4 links, 3 joints
Links:
- link base_link: geometry collision sphere radius=0.25; visual sphere radius=1.2

Commit message: Configure 6-drone area coverage simulation, optimal RRA return sweeps, and Gazebo 3D support

File: urdf/drone.urdf (robot description, URDF)
Before this commit: robot drone, 4 links, 3 joints
Links:
- link base_link: geometry collision sphere radius=0.25; visual box size=0.8 0.08 0.04
